Commit message: Adjust Panda URDF
Removed joint8 as it didn't serve any specific purpose and led to undesired collisions between joint7 and hand.
Converted visual meshes to convex collision meshes with vhacd.
Also cleaned up mesh files.

File: data/robots/panda/panda.urdf (robot description, URDF)
Before this commit: robot panda, 13 links, 12 joints
Links:
- removed link panda_link8
- link panda_link0: geometry collision mesh filename=package://meshes/collision/link0.obj; visual mesh filename=package://meshes/visual/link0.obj
- link panda_link7: geometry collision mesh filename=package://meshes/collision/link7.obj; visual mesh filename=package://meshes/visual/link7.obj
Joints:
- removed joint panda_joint8
- joint panda_hand_joint: origin xyz=0 0 0 rpy=0 0 -0.785398163397 -> xyz=0 0 0.107 rpy=0 0 -0.785398163397; parent panda_link8 -> panda_link7

Commit message: Add HER

File: data/robots/panda/panda.urdf (robot description, URDF)
Before this commit: robot panda, 12 links, 11 joints
Joints:
- joint panda_finger_joint2: mimic joint=panda_finger_joint1 -> (none)

Commit message: Resolve "Add UR5 robot"

File: data/robots/panda/panda.urdf (robot description, URDF)
Before this commit: robot panda, 12 links, 11 joints
Joints:
- joint panda_finger_joint2: limit lower=0.0 upper=0.04 effort=140 velocity=0.2 -> lower=0.0 upper=0.04 effort=140 velocity=0.0002
