Commit message: Add missing meshes

File: data/robots/ur5/ur5.urdf (robot description, URDF)
Before this commit: robot sisbot, 11 links, 10 joints
Links:
- removed link panda_grasptarget
- removed link panda_hand
- removed link panda_leftfinger
- removed link panda_rightfinger
- added link base, mass 0.0
- added link left_inner_finger, mass 0.00724255346165745; collision mesh filename=package://meshes/collision/inner_finger_coarse.STL; visual mesh filename=package://meshes/visual/inner_finger_fine.STL
- added link left_inner_knuckle, mass 0.0110930853895903; collision mesh filename=package://meshes/collision/inner_knuckle_coarse.STL; visual mesh filename=package://meshes/visual/inner_knuckle_fine.STL
- added link left_inner_loop, mass 0.0
- added link left_outer_finger, mass 0.0273093985570947; collision mesh filename=package://meshes/collision/outer_finger_coarse.STL; visual mesh filename=package://meshes/visual/outer_finger_fine.STL
- added link left_outer_knuckle, mass 0.00684838849434396; collision mesh filename=package://meshes/collision/outer_knuckle_coarse.STL; visual mesh filename=package://meshes/visual/outer_knuckle_fine.STL
- added link left_outer_loop, mass 0.0
- added link right_inner_finger, mass 0.00724255346165744; collision mesh filename=package://meshes/collision/inner_finger_coarse.STL; visual mesh filename=package://meshes/visual/inner_finger_fine.STL
- added link right_inner_knuckle, mass 0.0110930853895903; collision mesh filename=package://meshes/collision/inner_knuckle_coarse.STL; visual mesh filename=package://meshes/visual/inner_knuckle_fine.STL
- added link right_inner_loop, mass 0.0
- added link right_outer_finger, mass 0.0273093985570947; collision mesh filename=package://meshes/collision/outer_finger_coarse.STL; visual mesh filename=package://meshes/visual/outer_finger_fine.STL
- added link right_outer_knuckle, mass 0.00684838849401352; collision mesh filename=package://meshes/collision/outer_knuckle_coarse.STL; visual mesh filename=package://meshes/visual/outer_knuckle_fine.STL
- added link right_outer_loop, mass 0.0
- added link robotiq_85_base_link, mass 0.30915; collision mesh filename=package://meshes/collision/robotiq_85_base_link_coarse.STL; visual mesh filename=package://meshes/visual/robotiq_85_base_link_fine.STL
- added link tcp, mass 0.0
Joints:
- removed joint panda_finger_joint1
- removed joint panda_finger_joint2
- removed joint panda_grasptarget_hand
- removed joint panda_hand_joint
- added joint arm_gripper_joint: type fixed, parent wrist_3_link, child robotiq_85_base_link, origin xyz=0.0 0.0823 0.0 rpy=-1.570796 3.141592 0.0, axis 0 1 0
- added joint base_joint: type fixed, parent base, child base_link, origin xyz=0 0 0 rpy=0 0 1.570796, axis 0 -1 0
- added joint left_inner_finger_joint: type revolute, parent left_inner_knuckle, child left_inner_finger, origin xyz=0.034585310861294 0 0.0454970193817975 rpy=0 0 0, axis 0 -1 0, limit lower=0 upper=0.8757 effort=20 velocity=2.0
- added joint left_inner_finger_loop: type fixed, parent left_inner_finger, child left_inner_loop, origin xyz=0.018 0 -0.0065 rpy=0 0 0, axis 0 1 0, limit lower=-6.28318530718 upper=6.28318530718
- added joint left_inner_knuckle_joint: type revolute, parent robotiq_85_base_link, child left_inner_knuckle, origin xyz=0.0127000000001501 0 0.0693074999999639 rpy=0 0 0, axis 0 -1 0, limit lower=0 upper=0.8757 effort=20 velocity=2.0
- added joint left_outer_finger_joint: type fixed, parent left_outer_knuckle, child left_outer_finger, origin xyz=0.0316910442266543 0 -0.00193396375724605 rpy=0 0 0, axis 0 -1 0
- added joint left_outer_finger_loop: type fixed, parent left_outer_finger, child left_outer_loop, origin xyz=0.003 0 0.0475 rpy=0 0 0, axis 0 1 0
- added joint left_outer_knuckle_joint: type revolute, parent robotiq_85_base_link, child left_outer_knuckle, origin xyz=0.0306011444260539 0 0.0627920162695395 rpy=0 0 0, axis 0 -1 0, limit lower=0 upper=0.725 effort=20 velocity=2.0
- added joint right_inner_finger_joint: type revolute, parent right_inner_knuckle, child right_inner_finger, origin xyz=0.0341060475457406 0 0.0458573878541688 rpy=0 0 0, axis 0 -1 0, limit lower=0 upper=0.8757 effort=20 velocity=2.0
- added joint right_inner_finger_loop: type fixed, parent right_inner_finger, child right_inner_loop, origin xyz=0.018 0 -0.0065 rpy=0 0 0, axis 0 -1 0, limit lower=-6.28318530718 upper=6.28318530718
- added joint right_inner_knuckle_joint: type revolute, parent robotiq_85_base_link, child right_inner_knuckle, origin xyz=-0.0126999999998499 0 0.0693075000000361 rpy=0 0 3.14159265358979, axis 0 -1 0, limit lower=0 upper=0.8757 effort=20 velocity=2.0
- added joint right_outer_finger_joint: type fixed, parent right_outer_knuckle, child right_outer_finger, origin xyz=0.0317095909367246 0 -0.0016013564954687 rpy=0 0 0, axis 0 -1 0
- added joint right_outer_finger_loop: type fixed, parent right_outer_finger, child right_outer_loop, origin xyz=0.003 0 0.0475 rpy=0 0 0, axis 0 -1 0
- added joint right_outer_knuckle_joint: type revolute, parent robotiq_85_base_link, child right_outer_knuckle, origin xyz=-0.0306011444258893 0 0.0627920162695395 rpy=0 0 3.14159265358979, axis 0 -1 0, limit lower=0 upper=0.8757 effort=20 velocity=2.0
- added joint tcp: type fixed, parent robotiq_85_base_link, child tcp, origin xyz=0.0 0.0 0.15 rpy=0 0 -1.570796, axis 0 1 0
