Commit message: Create robot arm super class

File: karolos/environments/robot_task_environments/robots/Panda/panda.urdf (robot description, URDF)
Before this commit: robot panda, 12 links, 11 joints
Links:
- removed link panda_grasptarget
- added link tcp, mass 0.0
Joints:
- removed joint panda_grasptarget_hand
- added joint tcp: type fixed, parent panda_hand, child tcp, origin xyz=0 0 0.105 rpy=0 0 0

File: karolos/environments/robot_task_environments/robots/UR5/ur5.urdf (robot description, URDF)
Before this commit: robot ur5, 22 links, 21 joints
Links:
- removed link left_inner_knuckle
- removed link left_inner_loop
- removed link left_outer_finger
- removed link left_outer_knuckle
- removed link left_outer_loop
- removed link right_inner_knuckle
- removed link right_inner_loop
- removed link right_outer_finger
- removed link right_outer_knuckle
- removed link right_outer_loop
Joints:
- removed joint left_inner_finger_loop
- removed joint left_inner_knuckle_joint
- removed joint left_outer_finger_joint
- removed joint left_outer_finger_loop
- removed joint left_outer_knuckle_joint
- removed joint right_inner_finger_loop
- removed joint right_inner_knuckle_joint
- removed joint right_outer_finger_joint
- removed joint right_outer_finger_loop
- removed joint right_outer_knuckle_joint
- joint left_inner_finger_joint: axis 0 -1 0 -> -0.95307293 0. 0.30274081; limit lower=0 upper=0.8757 effort=20 velocity=2.0 -> lower=-.0425 upper=0. effort=10 velocity=0.1; origin xyz=0.034585310861294 0 0.0454970193817975 rpy=0 0 0 -> xyz=0.0064 0 0.126 rpy=0 0 0; parent left_inner_knuckle -> robotiq_85_base_link; type revolute -> prismatic
- joint right_inner_finger_joint: axis 0 -1 0 -> -0.95307293 0. 0.30274081; limit lower=0 upper=0.8757 effort=20 velocity=2.0 -> lower=-.0425 upper=0. effort=10 velocity=0.1; origin xyz=0.0341060475457406 0 0.0458573878541688 rpy=0 0 0 -> xyz=-0.0064 0 0.126 rpy=0 0 3.1416; parent right_inner_knuckle -> robotiq_85_base_link; type revolute -> prismatic

Commit message: Disable fingers and use fixed constraint instead to make gripping more robust

File: karolos/environments/robot_task_environments/robots/Panda/panda.urdf (robot description, URDF)
Before this commit: robot panda, 12 links, 11 joints
Joints:
- joint tcp: origin xyz=0 0 0.105 rpy=0 0 0 -> xyz=0 0 0.105 rpy=3.14159 0 0
