Commit message: Extend pick_place controller to UR5 robot

File: karolos/environments/robot_task_environments/robots/UR5/ur5.urdf (robot description, URDF)
Before this commit: robot ur5, 12 links, 11 joints
Joints:
- joint left_inner_finger_joint: axis -0.95307293 0. 0.30274081 -> 0.95307293 0. -0.30274081; limit lower=-.0425 upper=0. effort=10 velocity=0.1 -> lower=0. upper=.0425 effort=10 velocity=0.1
- joint right_inner_finger_joint: axis -0.95307293 0. 0.30274081 -> 0.95307293 0. -0.30274081; limit lower=-.0425 upper=0. effort=10 velocity=0.1 -> lower=0. upper=.0425 effort=10 velocity=0.1
- joint tcp: origin xyz=0.0 0.0 0.15 rpy=0 0 -1.570796 -> xyz=0.0 0.0 0.15 rpy=3.14159 0 -1.570796

Commit message: Adjust UR5 tcp

File: karolos/environments/robot_task_environments/robots/UR5/ur5.urdf (robot description, URDF)
Before this commit: robot ur5, 12 links, 11 joints
Joints:
- joint elbow_joint: limit lower=-3.14159265359 upper=3.14159265359 effort=300.0 velocity=3.15 -> lower=0 upper=3.14159265359 effort=300.0 velocity=3.15
