Commit message: Update robots
Remove WIP status from IIWA
Change DHT notation
Adjust urdf files to match DHT for Panda & UR5

File: karolos/environments/environments_robot_task/robots/Panda/panda.urdf (robot description, URDF)
Before this commit: robot panda, 12 links, 11 joints
Joints:
- joint panda_joint7: origin xyz=0.088 0 0 rpy=1.57079632679 0 0 -> xyz=0.088 0 0 rpy=1.57079632679 -0.785398163397 0

File: karolos/environments/environments_robot_task/robots/UR5/ur5.urdf (robot description, URDF)
Before this commit: robot ur5, 12 links, 11 joints
Links:
- removed link base
Joints:
- removed joint base_joint
- joint shoulder_lift_joint: origin xyz=0.0 0.13585 0.0 rpy=0.0 0.0 0.0 -> xyz=0.0 0.13585 0.0 rpy=0.0 1.5708 0.0
- joint wrist_1_joint: origin xyz=0.0 0.0 0.39225 rpy=0.0 0.0 0.0 -> xyz=0.0 0.0 0.39225 rpy=0.0 1.5708 0.0

Commit message: Adjust robots - Make action space dict - Introduce forcing of resets - Switch to fixed fingers

File: karolos/environments/environments_robot_task/robots/Panda/panda.urdf (robot description, URDF)
Before this commit: robot panda, 12 links, 11 joints
Joints:
- joint panda_finger_joint1: origin xyz=0 0 0.0584 rpy=0 0 0 -> xyz=0 0.04 0.0584 rpy=0 0 0; type prismatic -> fixed
- joint panda_finger_joint2: origin xyz=0 0 0.0584 rpy=0 0 0 -> xyz=0 -0.04 0.0584 rpy=0 0 0; type prismatic -> fixed

File: karolos/environments/environments_robot_task/robots/UR5/ur5.urdf (robot description, URDF)
Before this commit: robot ur5, 11 links, 10 joints
Joints:
- joint left_inner_finger_joint: origin xyz=0.0064 0 0.126 rpy=0 0 0 -> xyz=0.04 0 0.126 rpy=0 0 0; type prismatic -> fixed
- joint right_inner_finger_joint: origin xyz=-0.0064 0 0.126 rpy=0 0 3.1416 -> xyz=-0.04 0 0.126 rpy=0 0 3.1416; type prismatic -> fixed
